File: projects/MCU_datalogger/MCU_datalogger.kicad_pcb (KiCad board)
At the start: 2 copper layers, 50.8 x 35.5 mm, 33 parts, among them J1 Conn_01x04_Pin, J2 Conn_01x09_Pin, J3 Conn_01x04_Pin, J4 Conn_02x03_Odd_Even, U1 24LC1025, U2 DS1337S_, U3 24LC1025, U4 ATMEGA328P-AU, Y1 32.768KHz, Y2 16MHz

Commit message: MCU datalogger v2.1 (4-layer) complete, export gerbers
Routing:
- net /Vcc: track 141.5 -> 58.6 mm, vias 4 -> 15
- net GND: track 47.7 -> 36.8 mm, vias 12 -> 14
- net /SCK: track 91.8 -> 87.4 mm, vias 0 -> 3
- net Net-(U4-PB7): track 27.8 -> 24.1 mm
- net /D3: track 29.5 -> 26.1 mm
- net /D2: track 32.8 -> 29.8 mm
- net /D4: track 27.0 -> 24.2 mm
- net /SDA: track 65.2 -> 67.9 mm, vias 4 -> 3
- net /MISO: track 16.2 -> 18.4 mm, vias 2 -> 1
- net Net-(U4-AREF): track 9.56 -> 11.4 mm
- net /MOSI: track 18.5 -> 19.5 mm, vias 2 -> 0
- net Net-(U2-~{INTA}): track 7.60 -> 6.62 mm
- net /D8: track 12.3 -> 12.8 mm
- net /RESET: track 25.5 -> 25.9 mm, vias 3 -> 4
- net /TX: vias 2 -> 1
- added copper zone on In2.Cu, net /Vcc
- removed copper zone on F.Cu, net /Vcc
Other:
- copper layers 2 -> 4
- board text added: "MCU datalogger 4 layers v2.1"
- board text removed: "MCU datalogger 2 layers v1.2"

Commit message: MCU datalogger v2.1 (4-layer) - update PBC from schematic to bring /MH net label
Connections:
- net Net-(U4-AREF) renamed /MH
Changed lines of the file:
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@@
 	(net 3 "Net-(U4-PB6)")
 	(net 4 "Net-(U4-PB7)")
-	(net 5 "Net-(U4-AREF)")
+	(net 5 "/MH")
 	(net 6 "Net-(D1-K)")
 	(net 7 "/SCK")
@@
 			(layers "F.Cu" "F.Mask" "F.Paste")
 			(roundrect_rratio 0.125)
-			(net 5 "Net-(U4-AREF)")
+			(net 5 "/MH")
 			(pinfunction "AREF")
 			(pintype "input")
@@
 			(layers "F.Cu" "F.Mask" "F.Paste")
 			(roundrect_rratio 0.188679)
-			(net 5 "Net-(U4-AREF)")
+			(net 5 "/MH")
 			(pintype "passive")
 		)

Commit message: MCU datalogger v2.2 (4-layer) complete - fixes SCL/SCK bug
Connections:
- J1 pad 4: /SCK -> /SCL
- R2 pad 2: /SCK -> /SCL
- U1 pad 6: /SCK -> /SCL
- U2 pad 6: /SCK -> /SCL
- U3 pad 6: /SCK -> /SCL
- U4 pad 28: /SCK -> /SCL
Routing:
- net /SCL: track 0.00 -> 66.3 mm, vias 0 -> 3
- net /SCK: track 87.4 -> 23.9 mm, vias 3 -> 1
- net /MH: track 11.4 -> 12.6 mm
Other:
- board text added: "MCU datalogger 4 layers v2.2"
- board text removed: "MCU datalogger 4 layers v2.1"
