File: projects/pico_IoT_thingy/pico_IoT_thingy.kicad_pcb (KiCad board)
At the start: 4 copper layers, 95 x 75 mm, 61 parts, among them IC1 THVD1406DR, J1 Barrel_Jack_Switch, J2 QWIIC, J3 Conn_01x03, J4 Screw_Terminal_01x03, J5 Screw_Terminal_01x04, J6 Conn_02x05_Odd_Even, J7 Conn_01x02, K1 RT314A05, Q1 BC817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

Commit message: pico_IoT_thingy v1.3 Initial commit - fixes after testing 1st proto
Parts:
- moved C1 57.6 mm to (139.6, 81.9)
- moved C2 57.6 mm to (173.1, 127.7)
- moved C3 57.6 mm to (169.1, 127.7)
- moved C4 57.6 mm to (143.6, 75.9)
- moved C5 57.6 mm to (169.1, 121.7)
- moved C6 57.6 mm to (173.1, 121.7)
- moved D1 57.6 mm to (169.1, 136.5)
- moved D7 57.6 mm to (144.6, 124.3)
- moved D8 57.6 mm to (148.1, 132.5)
- moved F1 57.6 mm to (178.1, 136.5)
- moved H2 57.6 mm to (187.1, 70.5)
- moved H4 57.6 mm to (187.1, 137.5)
- moved IC1 57.6 mm to (136.1, 118.5)
- moved J2 57.6 mm to (139.6, 70.0)
- moved J7 57.6 mm to (149.1, 138.5)
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Routing:
- net +3V3: track 44.7 -> 34.2 mm, vias 19 -> 23
- net GND: track 99.2 -> 91.0 mm, vias 24 -> 26
- net Net-(F1-Pad1): track 10.7 -> 11.9 mm
- net /UART0_TX: track 40.6 -> 41.4 mm
- net /A: track 43.3 -> 42.4 mm
Other:
- board text added: "24VDC"
- board text added: "CS"
- board text added: "GPIO26"
- board text added: "GPIO27"
- board text added: "Raspberry Pi Pico IoT board with QWIIC and RS485 interfaces v1.3"
- board text added: "Rx"
- board text added: "SCK"
- board text added: "Tx"
- board text added: "Vcc"
