File: projects/pico_IoT_thingy/pico_IoT_thingy.kicad_sch (KiCad schematic)
At the start: 58 parts, among them IC1 THVD1406DR, J1 Barrel_Jack_Switch, J2 QWIIC, J3 Conn_01x03, J4 Screw_Terminal_01x03, J5 Screw_Terminal_01x04, J6 Conn_02x05_Odd_Even, J7 Conn_01x02, K1 RT314A05, Q1 BC817, SW1 SW_SPST, SW2 SW_SPST, SW3 SW_DIP_x04, U1 TSR_1-2450, U2 SHT31-DIS, U3 TLV1117-33

Commit message: Pico IoT thingy - logos and initial routing
Parts:
- A1, D3, D5, D8, J2, J3, J4, J5: Mouser Ref (none) -> aliexpress
- C1, C3, C4, C5, C6, C7, C8, D2, D4, J1, J7, R1, R10, R11, R12, R13, R14, R15, R16, R17, R18, R19, R2, R20, R3, R4, R5, R6, R7, R8, R9, SW1, SW2: Mouser Ref (none) -> stash
- C2: Mouser Ref (none) -> 581-12065C225K4Z2A
- D1: Mouser Ref (none) -> 576-SMAJ24A
- D7: Mouser Ref (none) -> 576-SM712-02HTG
- F1: Mouser Ref (none) -> 652-MFSM100-2
- H1, H2, H3, H4, JP1: Mouser Ref (none) -> na
- IC1: Mouser Ref (none) -> 595-THVD1406DR
- J6: Mouser Ref (none) -> 200-MTSW10509GD490
- K1: Mouser Ref (none) -> 655-RT314A05
- Q1: Mouser Ref (none) -> 583-BC817
- SW3: Mouser Ref (none) -> 774-2194MST
- U1: Mouser Ref (none) -> 495-TSR1-2450E
- U2: Mouser Ref (none) -> 403-SHT31ADIS-B2.5KS
- U3: Mouser Ref (none) -> 595-TLV1117-33IDCYR
Connections:
- net LOAD_COM: now reaches J4.2 (Pin_2), K1.11
- net LOAD_NC: now reaches J4.1 (Pin_1), K1.12
- net LOAD_NO: now reaches J4.3 (Pin_3), K1.14
Other:
- moved on the sheet: J4

Commit message: Pico IoT thingy v1.0 complete
Connections:
- net GND: no longer H2.1
- no-connect marks 12 -> 13
Other:
- note added: "Mounting Hole inside High Power area"
Changed lines of the file:
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@@
 	(title_block
 		(title "Pico IoT thingy")
-		(date "2026-01-05")
+		(date "2026-01-27")
 		(rev "1.0")
 		(company "Manuel Heredia")
@@
 		)
 	)
+	(text "Mounting Hole \ninside High Power area"
+		(exclude_from_sim no)
+		(at 190.5 49.53 0)
+		(effects
+			(font
+				(size 1.27 1.27)
+			)
+		)
+	)
 	(text "Extra GPIO pins \nfor the SPI port"
 		(exclude_from_sim no)
@@
 	)
 	(no_connect
+		(at 190.5 44.45)
+	)
+	(no_connect
 		(at 184.15 113.03)
 	)
@@
 	(symbol
 		(lib_id "power:GND")
-		(at 190.5 44.45 0)
+		(at 241.3 44.45 0)
 		(unit 1)
 		(exclude_from_sim no)
@@
 		(dnp no)
 		(property "Reference" "#PWR010"
-			(at 190.5 50.8 0)
+			(at 241.3 50.8 0)
 			(effects
 				(font
@@
 		)
 		(property "Value" "GND"
-			(at 190.5 48.26 0)
+			(at 241.3 48.26 0)
 			(effects
 				(font
@@
 		)
 		(property "Footprint" ""
-			(at 190.5 44.45 0)
+			(at 241.3 44.45 0)
 			(effects
 				(font
@@
 		)
 		(property "Datasheet" ""
-			(at 190.5 44.45 0)
+			(at 241.3 44.45 0)
 			(effects
 				(font
@@
 		)
 		(property "Description" "Power symbol creates a global label with name \"GND\" , ground"
-			(at 190.5 44.45 0)
+			(at 241.3 44.45 0)
 			(effects
 				(font
@@
 					(unit 1)
 				)
-			)
-		)
-	)
-	(symbol
-		(lib_id "power:GND")
-		(at 241.3 44.45 0)
-		(unit 1)
-		(exclude_from_sim no)
-		(in_bom yes)
-		(on_board yes)
-		(dnp no)
-		(property "Reference" "#PWR012"
-			(at 241.3 50.8 0)
-			(effects
-				(font
-					(size 1.27 1.27)
-				)
-				(hide yes)
-			)
-		)
-		(property "Value" "GND"
-			(at 241.3 48.26 0)
-			(effects
-				(font
-					(size 1.27 1.27)
-				)
-			)
-		)
-		(property "Footprint" ""
-			(at 241.3 44.45 0)
-			(effects
-				(font
-					(size 1.27 1.27)
-				)
-				(hide yes)
-			)
-		)
-		(property "Datasheet" ""
-			(at 241.3 44.45 0)
-			(effects
-				(font
-					(size 1.27 1.27)
-				)
-				(hide yes)
-			)
-		)
-		(property "Description" "Power symbol creates a global label with name \"GND\" , ground"
-			(at 241.3 44.45 0)
-			(effects
-				(font
-					(size 1.27 1.27)
-				)
-				(hide yes)
-			)
-		)
-		(pin "1"
-		)
-		(instances
-			(project "pico_IoT_thingy"
-				(path "/976a870b-4bc8-4381-8f7b-7356f08e7273"
-					(reference "#PWR012")
-					(unit 1)
-				)

Commit message: pico_IoT_thingy v1.3 Initial commit - fixes after testing 1st proto
Parts:
- D1: Height 2.29 -> (none); Manufacturer_Name Bourns -> (none); Manufacturer_Part_Number SMAJ24A -> (none); Mouser Part Number 652-SMAJ24A -> (none); Mouser Price/Stock https://www.mouser.co.uk/ProductDetail/Bourns/SMAJ24A?qs=A3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 -> (none)
- IC1: Height 1.75 -> (none); Manufacturer_Name Texas Instruments -> (none); Manufacturer_Part_Number THVD1406DR -> (none); Mouser Part Number 595-THVD1406DR -> (none); Mouser Price/Stock https://www.mouser.co.uk/ProductDetail/Texas-Instruments/TH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 -> (none)
- J3: Mouser Ref aliexpress -> stash
- J6: Mouser Ref 200-MTSW10509GD490 -> stash
- SW1, SW2: Mouser Ref stash -> aliexpress
Changed lines of the file:
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@@
 			)
 		)
-		(property "Mouser Ref" "aliexpress"
+		(property "Mouser Ref" "stash"
 			(at 171.45 88.9 0)
 			(effects
@@
 			)
 		)
-		(property "Height" "2.29"
-			(at -335.23 60.96 0)
-			(effects
-				(font
-					(size 1.27 1.27)
-				)
-				(justify left bottom)
-				(hide yes)
-			)
-		)
-		(property "Mouser Part Number" "652-SMAJ24A"
-			(at -435.23 60.96 0)
-			(effects
-				(font
-					(size 1.27 1.27)
-				)
-				(justify left bottom)
-				(hide yes)
-			)
-		)
-		(property "Mouser Price/Stock" "https://www.mouser.co.uk/ProductDetail/Bourns/SMAJ24A?qs=A3H9pljuJ8RK3%2FFerHGtzA%3D%3D"
-			(at -535.23 60.96 0)
-			(effects
-				(font
-					(size 1.27 1.27)
-				)
-				(justify left bottom)
-				(hide yes)
-			)
-		)
-		(property "Manufacturer_Name" "Bourns"
-			(at -635.23 60.96 0)
-			(effects
-				(font
-					(size 1.27 1.27)
-				)
-				(justify left bottom)
-				(hide yes)
-			)
-		)
-		(property "Manufacturer_Part_Number" "SMAJ24A"
-			(at -735.23 60.96 0)
-			(effects
-				(font
-					(size 1.27 1.27)
-				)
-				(justify left bottom)
-				(hide yes)
-			)
-		)
 		(property "Mouser Ref" " 576-SMAJ24A "
 			(at 58.42 50.8 90)
@@
 			)
 		)
-		(property "Mouser Ref" "200-MTSW10509GD490 "
+		(property "Mouser Ref" "stash"
 			(at 346.71 226.06 0)
 			(effects
@@
 			)
 		)
-		(property "Mouser Ref" "stash"
+		(property "Mouser Ref" "aliexpress"
 			(at 54.61 162.56 0)
 			(effects
@@
 			)
 		)
-		(property "Mouser Ref" "stash"
+		(property "Mouser Ref" "aliexpress"
 			(at 167.64 110.49 0)
 			(effects
@@
 				(hide yes)
 			)
-		)
-		(property "Height" "1.75"
-			(at 209.55 645.11 0)
-			(effects
-				(font
-					(size 1.27 1.27)
-				)
-				(justify left top)
-				(hide yes)
-			)
-		)
-		(property "Mouser Part Number" "595-THVD1406DR"
-			(at 209.55 745.11 0)
-			(effects
-				(font
-					(size 1.27 1.27)
-				)
-				(justify left top)
-				(hide yes)
-			)
-		)
-		(property "Mouser Price/Stock" "https://www.mouser.co.uk/ProductDetail/Texas-Instruments/THVD1406DR?qs=Li%252BoUPsLEnsDRatqPHNy8w%3D%3D"
-			(at 209.55 845.11 0)
-			(effects
-				(font
-					(size 1.27 1.27)
-				)
-				(justify left top)
-				(hide yes)
-			)
-		)
-		(property "Manufacturer_Name" "Texas Instruments"
-			(at 209.55 945.11 0)
-			(effects
-				(font
-					(size 1.27 1.27)
-				)
-				(justify left top)
-				(hide yes)
-			)
-		)
-		(property "Manufacturer_Part_Number" "THVD1406DR"
-			(at 209.55 1045.11 0)
-			(effects
-				(font
-					(size 1.27 1.27)
-				)
-				(justify left top)
-				(hide yes)
-			)
