File: projects/06_pico_IoT_thingy/pico_IoT_thingy.kicad_pcb (KiCad board)
At the start: 4 copper layers, 95 x 75 mm, 61 parts, among them IC1 THVD1406DR, J1 Barrel_Jack_Switch, J2 QWIIC, J3 Conn_01x03, J4 Screw_Terminal_01x03, J5 Screw_Terminal_01x04, J6 Conn_02x05_Odd_Even, J7 Conn_01x02, K1 RT314A05, Q1 BC817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

Commit message: pico_IoT_thingy - v1.4 WIP: add notes and replace LED symbol on schematic, improve labels
Schematic:

- add notes on:
  - U1: input voltage nominal 12V and range 6.5-36V
  - JP1: effect on SH31 I2C address
  - IC1: tying SHDN and RE to HIGH to enable auto-direction of RS485 transceiver
  - J7: jumper to enable termination resistor
- D8: replace RBG LED symbol from RGBA to BGRA type

PCB:

* swap NO and NC labels
* add labels to SPI and SWD connectors
Connections:
- A1 pad 21: /LED_B -> /LED_R
- A1 pad 24: /LED_R -> /LED_B
- R11 pad 1: /LED_R -> /LED_B
- R13 pad 1: /LED_B -> /LED_R
Other:
- board text added: "12VDC"
- board text added: "A0|D26"
- board text added: "A1|D27"
- board text added: "Raspberry Pi Pico IoT board with QWIIC and RS485 interfaces v1.4"
- board text added: "SWCLK"
- board text added: "SWDIO"
- board text removed: "24VDC"
- board text removed: "GPIO26"
- board text removed: "GPIO27"
- board text removed: "Raspberry Pi Pico IoT board with QWIIC and RS485 interfaces v1.3"
