File: projects/06_pico_IoT_thingy/pico_IoT_thingy.kicad_sch (KiCad schematic)
At the start: 58 parts, among them IC1 THVD1406DR, J1 Barrel_Jack_Switch, J2 QWIIC, J3 Conn_01x03, J4 Screw_Terminal_01x03, J5 Screw_Terminal_01x04, J6 Conn_02x05_Odd_Even, J7 Conn_01x02, K1 RT314A05, Q1 BC817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

Commit message: pico_IoT_thingy - v1.4 WIP: add notes and replace LED symbol on schematic, improve labels
Schematic:

- add notes on:
  - U1: input voltage nominal 12V and range 6.5-36V
  - JP1: effect on SH31 I2C address
  - IC1: tying SHDN and RE to HIGH to enable auto-direction of RS485 transceiver
  - J7: jumper to enable termination resistor
- D8: replace RBG LED symbol from RGBA to BGRA type

PCB:

* swap NO and NC labels
* add labels to SPI and SWD connectors
Parts:
- D8: value LED_RGBA -> LED_BGRA; symbol Device:LED_RGBA -> Device:LED_BGRA
- renumbered R13 to R11, R11 to R13
Connections:
- net LED_B: now also A1.24 (GPIO18), R13.1; no longer A1.21 (GPIO16), R11.1
- net LED_R: now also A1.21 (GPIO16), R11.1; no longer A1.24 (GPIO18), R13.1
Other:
- note added: "6.5-36VDC input range (12V Nominal)"
- note added: "Aliexpress RGB LEDs are actually BGRA: Pin | Color --------- 1 | BLUE 2 | GREEN 3 | RED 4 | ANODE"
- note added: "I2C Address JP1 open to set ADDR LOW: 0x44 Solder JP1 to set ADDR HIGH: 0x45"
- note added: "J7 is jumper to connect termination resistor R14?"
- note added: "Should be a RT314005 instead!!"
- note added: "Tying ~{SHDN} and ~{RE} together to HIGH enables Auto-direction mode which allows controlling driver and receiver using the data input pin D"
- note removed: "?"
- note removed: "Not seen in documentation..."
- moved on the sheet: R11, R13
